Commit message: add world link for rviz

File: urdf/km_dolly.urdf (robot description, URDF)
Before this commit: robot km_dolly, 7 links, 6 joints
Links:
- removed link horizontal_laser_link
Joints:
- removed joint horizontal_laser_link_joint

Commit message: better odometry

File: urdf/km_dolly.urdf (robot description, URDF)
Before this commit: robot km_dolly, 6 links, 5 joints
Links:
- link left_km1: geometry visual mesh filename=package://km_dolly/stl/Keigan_Dolly_KM-1U_L_resized.stl
- link right_km1: geometry visual mesh filename=package://km_dolly/stl/Keigan_Dolly_KM-1U_R_resized.stl
Joints:
- joint left_km1_joint: origin xyz=-0.09 0 0.062 rpy=0 0 0 -> xyz=0 0 0 rpy=0 0 0
- joint left_wheel_joint: origin xyz=-0.03 0 0 rpy=0 0 0 -> xyz=0 0 0 rpy=0 0 0
- joint right_km1_joint: origin xyz=0.09 0 0.062 rpy=0 0 0 -> xyz=0 0 0 rpy=0 0 0
